File: Telemaque.sch (KiCad schematic (older format))
At the start: 63 parts, among them J1 Conn_01x01, J2 Conn_01x01, J3 Conn_01x01, J4 Conn_01x01, P1 CONN_01X03, P2 CONN_01X10, P3 SMA, P4 CONN_01X05, P5 SMA, U1 LMC6482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

Commit message: Add files via upload
Parts:
- added C13: 1uF, symbol CP
- added C14: 100nF, Capacitors_SMD:C_0805_HandSoldering, symbol C
- added J1, J2, J3, J4: Test_1P, symbol Conn_01x01
- added L1, L2: L_Core_Ferrite_Small, Inductors_SMD:L_0805_HandSoldering, symbol L_Core_Ferrite_Small
- added U5: MC78M05CDT, TO_SOT_Packages_SMD:TO-252-2Lead, symbol MC78M05CDT
- C1, C2, C9: footprint (none) -> Capacitors_SMD:C_0805_HandSoldering
- C10: renamed from C12; footprint (none) -> Capacitors_SMD:C_0805_HandSoldering
- C11: renamed from C10; footprint (none) -> Capacitors_SMD:C_0805_HandSoldering
- C12: renamed from C11; footprint (none) -> Capacitors_SMD:C_0805_HandSoldering
- C15: renamed from C13; footprint (none) -> Capacitors_SMD:C_0805_HandSoldering
- C16: renamed from C14; footprint (none) -> Capacitors_SMD:C_0805_HandSoldering
- C17: renamed from C15; footprint (none) -> Capacitors_SMD:C_0805_HandSoldering
- C18: renamed from C16; footprint (none) -> Capacitors_SMD:C_0805_HandSoldering
- C19: renamed from C17; footprint (none) -> Capacitors_SMD:C_0805_HandSoldering
- C20: renamed from C18; footprint (none) -> Capacitors_SMD:C_0805_HandSoldering
- C21: renamed from C19; footprint (none) -> Capacitors_SMD:C_0805_HandSoldering
- C22: renamed from C20; footprint (none) -> Capacitors_SMD:C_0805_HandSoldering
- C3: renamed from C4; footprint (none) -> Capacitors_SMD:C_0805_HandSoldering
- C4: renamed from C3; footprint (none) -> Capacitors_SMD:C_0805_HandSoldering
- C5: renamed from C7; footprint (none) -> Capacitors_SMD:C_0805_HandSoldering
- C6: renamed from C5; footprint (none) -> Capacitors_SMD:C_0805_HandSoldering
- C7: renamed from C8; footprint (none) -> Capacitors_Tantalum_SMD:CP_Tantalum_Case-A_EIA-3216-18_Hand
- C8: renamed from C6; value C -> 10nF; footprint (none) -> Capacitors_SMD:C_0805_HandSoldering
- D2, D3, D4, D5: footprint (none) -> Diodes_SMD:D_SOT-23_ANK
- P1: footprint (none) -> Connectors_Molex:Molex_KK-6410-03_03x2.54mm_Straight
- P2: footprint (none) -> Connectors_Molex:Molex_KK-6410-10_10x2.54mm_Straight
- P3, P5: footprint (none) -> SMA_PINS:SMA_PINS
- P4: footprint (none) -> Connectors_Molex:Molex_KK-6410-05_05x2.54mm_Straight
- R1, R10, R11, R12, R13, R16, R19, R2, R20, R21, R22, R23, R24, R3, R4, R5, R6, R9: footprint (none) -> Resistors_SMD:R_0805_HandSoldering
- R14, R15, R17, R18, R7, R8: footprint (none) -> Resistors_SMD:R_1206_HandSoldering
- U2: renamed from U1; footprint (none) -> Housings_SOIC:SO-8_5.3x6.2mm_Pitch1.27mm
- U4: renamed from U3; footprint (none) -> Housings_SOIC:SO-8_5.3x6.2mm_Pitch1.27mm
- U6: renamed from U5; footprint (none) -> Housings_SOIC:SO-8_5.3x6.2mm_Pitch1.27mm
- renumbered J1 to J5, J2 to J6, J3 to J7, J4 to J8, U2 to U1, U4 to U3
Connections:
- net labels added: +5VA, +5VD
- net labels removed: +5V, +8V
- wire segments 152 -> 170
Other:
- moved on the sheet: C10, C11, C12, C15, C3, C5, C7, C9, J5, J6, J7, J8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
