File: Telemaque.sch (KiCad schematic (older format))
At the start: 81 parts, among them J1 Test, J10 Conn_Coaxial, J11 Conn_Coaxial, J2 Test, J3 Test, J4 Test, J5 Conn_01x01, J6 Conn_01x01, J7 Conn_01x01, J8 Conn_Coaxial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

Commit message: Add files via upload
Parts:
- added P3: CONN_01X03, symbol CONN_01X03
Connections:
- net +12V: now also P3.1 (P1)
- net +5VA: no longer C2.1
- net GND: now also P3.2 (P2)
- net at P2.3 (P3): now also P3.3 (P3); no longer P4.5 (P5)
- net at L1.1, P1.1 (P1): now also C2.1
Other:
- note added: "+12V"
- note added: "TxRx"
- note added: "from ?"
- note removed: "TxRxRly"
- moved on the sheet: C2, C20, C23, L1
