File: Telemaque.kicad_pcb (KiCad board)
At the start: 2 copper layers, 100.4 x 50 mm, 75 parts, among them J1 Test, J2 Test, J3 Test, J4 Test, J5 Conn_01x01, J6 Conn_01x01, J7 Conn_01x01, P1 CONN_01X03, P2 CONN_01X10, P3 SMA, P4 CONN_01X05, P5 SMA, U1 LMC6482, U2 LD1117STR, U3 LD1117S50TR, U4 ACS723LLCTR-40AU-T, U5 LD1117S50TR, U6 LMC6482

Commit message: Add files via upload
Parts:
- removed P3, P5: SMA, SMA_PINS:SMA_EDGE_NRW
- added J10: Conn_Coaxial, SMA_PINS:SMA_PINS, F.Cu at (164.0, 125.0)
- added J11: Conn_Coaxial, SMA_PINS:SMA_EDGE_NRW, F.Cu at (164.0, 127.0)
- added J8: Conn_Coaxial, SMA_PINS:SMA_PINS, F.Cu at (147.0, 125.0)
- added J9: Conn_Coaxial, SMA_PINS:SMA_EDGE_NRW, F.Cu at (147.0, 127.0)
- added L5: L_Core_Ferrite_Small, Inductors_SMD:L_0805_HandSoldering, F.Cu at (159.5, 84.0)
- added R26: R, Resistors_SMD:R_0805_HandSoldering, F.Cu at (160.0, 94.5)
- added R27: R, Resistors_SMD:R_0805_HandSoldering, F.Cu at (172.0, 94.5)
- added U7: LMC6082, Housings_SOIC:SO-8_5.3x6.2mm_Pitch1.27mm, F.Cu at (166.0, 91.0)
- C10, C17, C18, C19, C21, C22, C23: footprint Capacitors_SMD:C_0805_HandSoldering -> Resistors_SMD:R_0805_HandSoldering
- C6, C8: footprint Capacitors_SMD:C_0805_HandSoldering -> Capacitors_SMD:C_1206_HandSoldering
- J2: moved to F.Cu
- R1: value 2K -> R
- U4: footprint Housings_SOIC:SOIC-8_3.9x4.9mm_Pitch1.27mm -> Housings_SOIC:SO-8_5.3x6.2mm_Pitch1.27mm
- moved J2 92.6 mm to (85.0, 85.0)
- moved J3 92.6 mm to (85.0, 125.0)
- moved J1 87.5 mm to (175.0, 85.0)
- moved J4 87.5 mm to (175.0, 125.0)
- moved C1 45.9 mm to (166.0, 84.0)
- moved C4 25.0 mm to (123.7, 89.5), turned to 90 degrees
- moved C12 23.3 mm to (104.3, 113.4), turned to 270 degrees
- moved C3 17.4 mm to (132.0, 98.0)
- moved C7 14.4 mm to (116.0, 100.5), turned to 90 degrees
- moved C8 13.4 mm to (96.0, 115.2)
- moved U3 13.1 mm to (113.0, 115.0), turned to 180 degrees
- moved U1 11.2 mm to (91.0, 106.0)
- moved R7 10.8 mm to (99.0, 111.0)
- moved R4 10.6 mm to (84.0, 105.0)
- moved R3 9.89 mm to (120.0, 106.0), turned to 0 degrees
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Connections:
- C1 pad 1: +12V -> Net-(C1-Pad1)
- P2 pad 10: GND -> Net-(P2-Pad10)
- P2 pad 9: Net-(P2-Pad9) -> GND
- R1 pad 1: Net-(P2-Pad9) -> Net-(P1-Pad3)
- R1 pad 2: Net-(P1-Pad3) -> Net-(P2-Pad10)
Routing:
- net Net-(P2-Pad10): track 0.00 -> 97.8 mm, vias 0 -> 1
- net Net-(P2-Pad9): track 94.5 -> 0.00 mm, vias 1 -> 0
- net +5VA: track 43.0 -> 114.7 mm, vias 2 -> 3
- net Net-(C13-Pad1): track 55.7 -> 38.8 mm
- net Net-(R26-Pad1): track 0.00 -> 16.8 mm
- net Net-(P2-Pad3): track 18.8 -> 2.25 mm
- net Net-(P1-Pad3): track 3.51 -> 17.7 mm
- net Net-(J5-Pad1): track 73.6 -> 59.4 mm
- net Net-(P2-Pad7): track 19.7 -> 29.9 mm
- net Net-(P2-Pad6): track 20.0 -> 29.8 mm
- net Net-(J6-Pad1): track 50.7 -> 41.4 mm
- net Net-(D2-Pad2): track 26.7 -> 19.5 mm
- net Net-(C1-Pad1): track 0.00 -> 6.62 mm
- net Net-(D3-Pad1): track 10.7 -> 17.2 mm
- net Net-(C23-Pad1): track 74.1 -> 80.1 mm
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- added copper zone on B.Cu, net GND
Other:
- board size 100.4 x 50 mm -> 100 x 50 mm

Commit message: Add files via upload
Parts:
- added REF**: via, via:via, F.Cu at (159.0, 128.0)
- added REF**: via, via:via, F.Cu at (158.0, 127.0)
- added REF**: via, via:via, F.Cu at (178.0, 112.0)
- added REF**: via, via:via, F.Cu at (178.0, 111.0)
- added REF**: via, via:via, F.Cu at (178.0, 110.0)
- added REF**: via, via:via, F.Cu at (178.0, 109.0)
- added REF**: via, via:via, F.Cu at (178.0, 108.0)
- added REF**: via, via:via, F.Cu at (178.0, 107.0)
- added REF**: via, via:via, F.Cu at (178.0, 106.0)
- added REF**: via, via:via, F.Cu at (178.0, 105.0)
- added REF**: via, via:via, F.Cu at (178.0, 104.0)
- added REF**: via, via:via, F.Cu at (178.0, 103.0)
- added REF**: via, via:via, F.Cu at (157.0, 127.0)
- added REF**: via, via:via, F.Cu at (178.0, 102.0)
- added REF**: via, via:via, F.Cu at (178.0, 101.0)
- added REF**: via, via:via, F.Cu at (178.0, 100.0)
- added REF**: via, via:via, F.Cu at (178.0, 99.0)
- added REF**: via, via:via, F.Cu at (178.0, 98.0)
- added REF**: via, via:via, F.Cu at (178.0, 97.0)
- added REF**: via, via:via, F.Cu at (178.0, 96.0)
- added REF**: via, via:via, F.Cu at (178.0, 95.0)
- added REF**: via, via:via, F.Cu at (178.0, 94.0)
- added REF**: via, via:via, F.Cu at (178.0, 93.0)
- added REF**: via, via:via, F.Cu at (156.0, 127.0)
- added REF**: via, via:via, F.Cu at (178.0, 92.0)
- added REF**: via, via:via, F.Cu at (178.0, 91.0)
- added REF**: via, via:via, F.Cu at (178.0, 90.0)
- added REF**: via, via:via, F.Cu at (142.0, 128.0)
- added REF**: via, via:via, F.Cu at (141.0, 128.0)
- added REF**: via, via:via, F.Cu at (140.0, 128.0)
- added REF**: via, via:via, F.Cu at (139.0, 128.0)
- added REF**: via, via:via, F.Cu at (138.0, 128.0)
- added REF**: via, via:via, F.Cu at (137.0, 128.0)
- added REF**: via, via:via, F.Cu at (136.0, 128.0)
- added REF**: via, via:via, F.Cu at (155.0, 127.0)
- added REF**: via, via:via, F.Cu at (135.0, 128.0)
- added REF**: via, via:via, F.Cu at (134.0, 128.0)
- added REF**: via, via:via, F.Cu at (133.0, 128.0)
- added REF**: via, via:via, F.Cu at (132.0, 128.0)
- added REF**: via, via:via, F.Cu at (131.0, 128.0)
- added REF**: via, via:via, F.Cu at (130.0, 128.0)
- added REF**: via, via:via, F.Cu at (129.0, 128.0)
- added REF**: via, via:via, F.Cu at (128.0, 128.0)
- added REF**: via, via:via, F.Cu at (127.0, 128.0)
- added REF**: via, via:via, F.Cu at (126.0, 128.0)
- added REF**: via, via:via, F.Cu at (154.0, 127.0)
- added REF**: via, via:via, F.Cu at (125.0, 128.0)
- added REF**: via, via:via, F.Cu at (124.0, 128.0)
- added REF**: via, via:via, F.Cu at (123.0, 128.0)
- added REF**: via, via:via, F.Cu at (122.0, 128.0)
- added REF**: via, via:via, F.Cu at (121.0, 128.0)
- added REF**: via, via:via, F.Cu at (120.0, 128.0)
- added REF**: via, via:via, F.Cu at (119.0, 128.0)
- added REF**: via, via:via, F.Cu at (118.0, 128.0)
- added REF**: via, via:via, F.Cu at (117.0, 128.0)
- added REF**: via, via:via, F.Cu at (116.0, 128.0)
- added REF**: via, via:via, F.Cu at (153.0, 127.0)
- added REF**: via, via:via, F.Cu at (115.0, 128.0)
- added REF**: via, via:via, F.Cu at (114.0, 128.0)
- added REF**: via, via:via, F.Cu at (113.0, 128.0)
- added REF**: via, via:via, F.Cu at (112.0, 128.0)
- added REF**: via, via:via, F.Cu at (111.0, 128.0)
- added REF**: via, via:via, F.Cu at (110.0, 128.0)
- added REF**: via, via:via, F.Cu at (109.0, 128.0)
- added REF**: via, via:via, F.Cu at (108.0, 128.0)
- added REF**: via, via:via, F.Cu at (107.0, 128.0)
- added REF**: via, via:via, F.Cu at (106.0, 128.0)
- added REF**: via, via:via, F.Cu at (152.0, 127.0)
- added REF**: via, via:via, F.Cu at (105.0, 128.0)
- added REF**: via, via:via, F.Cu at (104.0, 128.0)
- added REF**: via, via:via, F.Cu at (103.0, 128.0)
- added REF**: via, via:via, F.Cu at (102.0, 128.0)
- added REF**: via, via:via, F.Cu at (101.0, 128.0)
- added REF**: via, via:via, F.Cu at (100.0, 128.0)
- added REF**: via, via:via, F.Cu at (99.0, 128.0)
- added REF**: via, via:via, F.Cu at (98.0, 128.0)
- added REF**: via, via:via, F.Cu at (97.0, 128.0)
- added REF**: via, via:via, F.Cu at (96.0, 128.0)
- added REF**: via, via:via, F.Cu at (159.0, 126.0)
- added REF**: via, via:via, F.Cu at (95.0, 128.0)
- added REF**: via, via:via, F.Cu at (94.0, 128.0)
- added REF**: via, via:via, F.Cu at (93.0, 128.0)
- added REF**: via, via:via, F.Cu at (92.0, 128.0)
- added REF**: via, via:via, F.Cu at (91.0, 128.0)
- added REF**: via, via:via, F.Cu at (90.0, 128.0)
- added REF**: via, via:via, F.Cu at (89.0, 128.0)
- added REF**: via, via:via, F.Cu at (178.0, 89.0)
- added REF**: via, via:via, F.Cu at (170.0, 82.0)
- added REF**: via, via:via, F.Cu at (169.0, 82.0)
- added REF**: via, via:via, F.Cu at (158.0, 126.0)
- added REF**: via, via:via, F.Cu at (168.0, 82.0)
- added REF**: via, via:via, F.Cu at (167.0, 82.0)
- added REF**: via, via:via, F.Cu at (166.0, 82.0)
- added REF**: via, via:via, F.Cu at (165.0, 82.0)
- added REF**: via, via:via, F.Cu at (164.0, 82.0)
- added REF**: via, via:via, F.Cu at (163.0, 82.0)
- added REF**: via, via:via, F.Cu at (162.0, 82.0)
- added REF**: via, via:via, F.Cu at (161.0, 82.0)
- added REF**: via, via:via, F.Cu at (160.0, 82.0)
- added REF**: via, via:via, F.Cu at (159.0, 82.0)
- added REF**: via, via:via, F.Cu at (157.0, 126.0)
- added REF**: via, via:via, F.Cu at (158.0, 82.0)
- added REF**: via, via:via, F.Cu at (157.0, 82.0)
- added REF**: via, via:via, F.Cu at (156.0, 82.0)
- added REF**: via, via:via, F.Cu at (155.0, 82.0)
- added REF**: via, via:via, F.Cu at (154.0, 82.0)
- added REF**: via, via:via, F.Cu at (153.0, 82.0)
- added REF**: via, via:via, F.Cu at (152.0, 82.0)
- added REF**: via, via:via, F.Cu at (151.0, 82.0)
- added REF**: via, via:via, F.Cu at (150.0, 82.0)
- added REF**: via, via:via, F.Cu at (149.0, 82.0)
- added REF**: via, via:via, F.Cu at (158.0, 128.0)
- added REF**: via, via:via, F.Cu at (156.0, 126.0)
- added REF**: via, via:via, F.Cu at (148.0, 82.0)
- added REF**: via, via:via, F.Cu at (147.0, 82.0)
- added REF**: via, via:via, F.Cu at (146.0, 82.0)
- added REF**: via, via:via, F.Cu at (145.0, 82.0)
- added REF**: via, via:via, F.Cu at (144.0, 82.0)
- added REF**: via, via:via, F.Cu at (143.0, 82.0)
- added REF**: via, via:via, F.Cu at (142.0, 82.0)
- added REF**: via, via:via, F.Cu at (141.0, 82.0)
- added REF**: via, via:via, F.Cu at (140.0, 82.0)
- added REF**: via, via:via, F.Cu at (139.0, 82.0)
- added REF**: via, via:via, F.Cu at (155.0, 126.0)
- added REF**: via, via:via, F.Cu at (138.0, 82.0)
- added REF**: via, via:via, F.Cu at (137.0, 82.0)
- added REF**: via, via:via, F.Cu at (136.0, 82.0)
- added REF**: via, via:via, F.Cu at (135.0, 82.0)
- added REF**: via, via:via, F.Cu at (134.0, 82.0)
- added REF**: via, via:via, F.Cu at (133.0, 82.0)
- added REF**: via, via:via, F.Cu at (132.0, 82.0)
- added REF**: via, via:via, F.Cu at (131.0, 82.0)
- added REF**: via, via:via, F.Cu at (130.0, 82.0)
- added REF**: via, via:via, F.Cu at (129.0, 82.0)
- added REF**: via, via:via, F.Cu at (154.0, 126.0)
- added REF**: via, via:via, F.Cu at (128.0, 82.0)
- added REF**: via, via:via, F.Cu at (127.0, 82.0)
- added REF**: via, via:via, F.Cu at (126.0, 82.0)
- added REF**: via, via:via, F.Cu at (125.0, 82.0)
- added REF**: via, via:via, F.Cu at (124.0, 82.0)
- added REF**: via, via:via, F.Cu at (123.0, 82.0)
- added REF**: via, via:via, F.Cu at (122.0, 82.0)
- added REF**: via, via:via, F.Cu at (121.0, 82.0)
- added REF**: via, via:via, F.Cu at (120.0, 82.0)
- added REF**: via, via:via, F.Cu at (119.0, 82.0)
- added REF**: via, via:via, F.Cu at (153.0, 126.0)
- added REF**: via, via:via, F.Cu at (118.0, 82.0)
- added REF**: via, via:via, F.Cu at (117.0, 82.0)
- added REF**: via, via:via, F.Cu at (116.0, 82.0)
- added REF**: via, via:via, F.Cu at (115.0, 82.0)
- added REF**: via, via:via, F.Cu at (114.0, 82.0)
- added REF**: via, via:via, F.Cu at (113.0, 82.0)
- added REF**: via, via:via, F.Cu at (112.0, 82.0)
- added REF**: via, via:via, F.Cu at (111.0, 82.0)
- added REF**: via, via:via, F.Cu at (110.0, 82.0)
- added REF**: via, via:via, F.Cu at (109.0, 82.0)
- added REF**: via, via:via, F.Cu at (83.0, 121.0)
- added REF**: via, via:via, F.Cu at (108.0, 82.0)
- added REF**: via, via:via, F.Cu at (107.0, 82.0)
- added REF**: via, via:via, F.Cu at (106.0, 82.0)
- added REF**: via, via:via, F.Cu at (105.0, 82.0)
- added REF**: via, via:via, F.Cu at (104.0, 82.0)
- added REF**: via, via:via, F.Cu at (103.0, 82.0)
- added REF**: via, via:via, F.Cu at (102.0, 82.0)
- added REF**: via, via:via, F.Cu at (101.0, 82.0)
- added REF**: via, via:via, F.Cu at (100.0, 82.0)
- added REF**: via, via:via, F.Cu at (99.0, 82.0)
- added REF**: via, via:via, F.Cu at (82.0, 121.0)
- added REF**: via, via:via, F.Cu at (98.0, 82.0)
- added REF**: via, via:via, F.Cu at (97.0, 82.0)
- added REF**: via, via:via, F.Cu at (96.0, 82.0)
- added REF**: via, via:via, F.Cu at (95.0, 82.0)
- added REF**: via, via:via, F.Cu at (94.0, 82.0)
- added REF**: via, via:via, F.Cu at (93.0, 82.0)
- added REF**: via, via:via, F.Cu at (92.0, 82.0)
- added REF**: via, via:via, F.Cu at (91.0, 82.0)
- added REF**: via, via:via, F.Cu at (90.0, 82.0)
- added REF**: via, via:via, F.Cu at (89.0, 82.0)
- added REF**: via, via:via, F.Cu at (83.0, 120.0)
- added REF**: via, via:via, F.Cu at (82.0, 120.0)
- added REF**: via, via:via, F.Cu at (83.0, 119.0)
- added REF**: via, via:via, F.Cu at (82.0, 119.0)
- added REF**: via, via:via, F.Cu at (157.0, 128.0)
- added REF**: via, via:via, F.Cu at (83.0, 118.0)
- added REF**: via, via:via, F.Cu at (82.0, 118.0)
- added REF**: via, via:via, F.Cu at (83.0, 117.0)
- added REF**: via, via:via, F.Cu at (82.0, 117.0)
- added REF**: via, via:via, F.Cu at (83.0, 116.0)
- added REF**: via, via:via, F.Cu at (82.0, 116.0)
- added REF**: via, via:via, F.Cu at (83.0, 115.0)
- added REF**: via, via:via, F.Cu at (82.0, 115.0)
- added REF**: via, via:via, F.Cu at (83.0, 114.0)
- added REF**: via, via:via, F.Cu at (82.0, 114.0)
- added REF**: via, via:via, F.Cu at (156.0, 128.0)
- added REF**: via, via:via, F.Cu at (83.0, 113.0)
- added REF**: via, via:via, F.Cu at (82.0, 113.0)
- added REF**: via, via:via, F.Cu at (83.0, 112.0)
- added REF**: via, via:via, F.Cu at (82.0, 112.0)
- added REF**: via, via:via, F.Cu at (83.0, 111.0)
- added REF**: via, via:via, F.Cu at (82.0, 111.0)
- added REF**: via, via:via, F.Cu at (83.0, 110.0)
- added REF**: via, via:via, F.Cu at (82.0, 110.0)
- added REF**: via, via:via, F.Cu at (83.0, 109.0)
- added REF**: via, via:via, F.Cu at (82.0, 109.0)
- added REF**: via, via:via, F.Cu at (155.0, 128.0)
- added REF**: via, via:via, F.Cu at (83.0, 108.0)
- added REF**: via, via:via, F.Cu at (82.0, 108.0)
- added REF**: via, via:via, F.Cu at (83.0, 107.0)
- added REF**: via, via:via, F.Cu at (82.0, 107.0)
- added REF**: via, via:via, F.Cu at (83.0, 106.0)
- added REF**: via, via:via, F.Cu at (82.0, 106.0)
- added REF**: via, via:via, F.Cu at (83.0, 105.0)
- added REF**: via, via:via, F.Cu at (82.0, 105.0)
- added REF**: via, via:via, F.Cu at (83.0, 104.0)
- added REF**: via, via:via, F.Cu at (82.0, 104.0)
- added REF**: via, via:via, F.Cu at (154.0, 128.0)
- added REF**: via, via:via, F.Cu at (83.0, 103.0)
- added REF**: via, via:via, F.Cu at (82.0, 103.0)
- added REF**: via, via:via, F.Cu at (83.0, 102.0)
- added REF**: via, via:via, F.Cu at (82.0, 102.0)
- added REF**: via, via:via, F.Cu at (83.0, 101.0)
- added REF**: via, via:via, F.Cu at (82.0, 101.0)
- added REF**: via, via:via, F.Cu at (83.0, 100.0)
- added REF**: via, via:via, F.Cu at (82.0, 100.0)
- added REF**: via, via:via, F.Cu at (83.0, 99.0)
- added REF**: via, via:via, F.Cu at (82.0, 99.0)
- added REF**: via, via:via, F.Cu at (153.0, 128.0)
- added REF**: via, via:via, F.Cu at (83.0, 98.0)
- added REF**: via, via:via, F.Cu at (82.0, 98.0)
- added REF**: via, via:via, F.Cu at (83.0, 97.0)
- added REF**: via, via:via, F.Cu at (82.0, 97.0)
- added REF**: via, via:via, F.Cu at (83.0, 96.0)
- added REF**: via, via:via, F.Cu at (82.0, 96.0)
- added REF**: via, via:via, F.Cu at (83.0, 95.0)
- added REF**: via, via:via, F.Cu at (82.0, 95.0)
- added REF**: via, via:via, F.Cu at (83.0, 94.0)
- added REF**: via, via:via, F.Cu at (82.0, 94.0)
- added REF**: via, via:via, F.Cu at (152.0, 128.0)
- added REF**: via, via:via, F.Cu at (83.0, 93.0)
- added REF**: via, via:via, F.Cu at (82.0, 93.0)
- added REF**: via, via:via, F.Cu at (83.0, 92.0)
- added REF**: via, via:via, F.Cu at (82.0, 92.0)
- added REF**: via, via:via, F.Cu at (83.0, 91.0)
- added REF**: via, via:via, F.Cu at (82.0, 91.0)
- added REF**: via, via:via, F.Cu at (83.0, 90.0)
- added REF**: via, via:via, F.Cu at (82.0, 90.0)
- added REF**: via, via:via, F.Cu at (83.0, 89.0)
- added REF**: via, via:via, F.Cu at (152.0, 126.0)
- added REF**: via, via:via, F.Cu at (159.0, 127.0)
- added REF**: via, via:via, F.Cu at (82.0, 89.0)
- added REF**: via, via:via, F.Cu at (178.0, 121.0)
- added REF**: via, via:via, F.Cu at (178.0, 120.0)
- added REF**: via, via:via, F.Cu at (178.0, 119.0)
- added REF**: via, via:via, F.Cu at (178.0, 118.0)
- added REF**: via, via:via, F.Cu at (178.0, 117.0)
- added REF**: via, via:via, F.Cu at (178.0, 116.0)
- added REF**: via, via:via, F.Cu at (178.0, 115.0)
- added REF**: via, via:via, F.Cu at (178.0, 114.0)
- added REF**: via, via:via, F.Cu at (178.0, 113.0)
- moved C20 14.9 mm to (134.0, 116.0), turned to 0 degrees
- moved R4 5.39 mm to (86.0, 100.0)
- moved R5 3.16 mm to (87.0, 114.0)
- moved C6 3.00 mm to (90.0, 114.0)
- moved D1 1.00 mm to (127.0, 114.0)
Routing:
- net GND: track 18.0 -> 278.8 mm, vias 0 -> 73
- net Net-(J6-Pad1): track 41.4 -> 68.6 mm
- net Net-(J5-Pad1): track 59.4 -> 79.4 mm
- net Net-(P2-Pad3): track 2.25 -> 17.9 mm
- net Net-(C13-Pad1): track 38.8 -> 48.1 mm
- net Net-(C6-Pad1): track 12.3 -> 18.5 mm
- net Net-(D2-Pad2): track 19.5 -> 25.0 mm
- net Net-(C3-Pad1): track 23.7 -> 29.1 mm, vias 0 -> 4
- net +12V: track 35.6 -> 40.8 mm
- net (no net): track 2.63 -> 0.00 mm
