File: Telemaque.kicad_pcb (KiCad board)
At the start: 2 copper layers, 100 x 50 mm, 340 parts, among them J1 Test, J10 Conn_Coaxial, J11 Conn_Coaxial, J2 Test, J3 Test, J4 Test, J5 Conn_01x01, J6 Conn_01x01, J7 Conn_01x01, J8 Conn_Coaxial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

Commit message: Add files via upload
Parts:
- added P3: CONN_01X03, Connectors_Molex:Molex_KK-6410-03_03x2.54mm_Straight, F.Cu at (161.5, 87.0)
- J1, J2, J3, J4: footprint Mounting_Holes:MountingHole_3.5mm -> Mounting_Holes:MountingHole_3.2mm_M3_ISO7380
- U7: value LMC6082 -> LMC6482
- moved R27 84.0 mm to (88.0, 92.0), turned to 180 degrees
- moved U7 78.3 mm to (88.5, 102.0), turned to 270 degrees
- moved C1 73.0 mm to (95.5, 103.0)
- moved R26 70.5 mm to (89.5, 95.0), turned to 0 degrees
- moved L5 67.7 mm to (95.5, 106.0), turned to 180 degrees
- moved R1 66.8 mm to (94.0, 99.0), turned to 90 degrees
- moved R4 10.5 mm to (85.0, 110.5)
- moved R7 7.81 mm to (105.0, 106.0), turned to 180 degrees
- moved C5 6.52 mm to (100.0, 104.5)
- moved R13 5.59 mm to (161.0, 95.0), turned to 0 degrees
- moved U1 5.59 mm to (92.0, 111.5)
- moved R5 5.02 mm to (86.5, 119.0), turned to 0 degrees
- moved L2 5.00 mm to (99.0, 110.5)
- moved C6 4.30 mm to (86.5, 116.5), turned to 0 degrees
- moved L1 3.26 mm to (144.2, 88.8), turned to 270 degrees
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Connections:
- C2 pad 1: +5VA -> Net-(C2-Pad1)
- L1 pad 1: Net-(L1-Pad1) -> Net-(C2-Pad1)
- P1 pad 1: Net-(L1-Pad1) -> Net-(C2-Pad1)
- P4 pad 5: Net-(P2-Pad3) -> Net-(P4-Pad5)
Routing:
- net Net-(P1-Pad3): track 17.7 -> 83.8 mm, vias 0 -> 1
- net Net-(P2-Pad10): track 97.8 -> 36.8 mm
- net Net-(P2-Pad3): track 17.9 -> 78.4 mm
- net +12V: track 40.8 -> 82.6 mm
- net GND: track 278.8 -> 237.2 mm, vias 73 -> 44
- net +5VA: track 114.7 -> 90.6 mm, vias 3 -> 4
- net Net-(J5-Pad1): track 79.4 -> 95.0 mm
- net Net-(C8-Pad1): track 11.9 -> 20.8 mm
- net Net-(R26-Pad1): track 16.8 -> 7.86 mm
- net Net-(C2-Pad1): track 0.00 -> 7.32 mm
- net Net-(C10-Pad2): track 13.8 -> 6.97 mm
- net Net-(C6-Pad1): track 18.5 -> 11.8 mm
- net Net-(P2-Pad7): track 29.9 -> 23.6 mm
- net Net-(C23-Pad1): track 80.1 -> 75.4 mm
- net Net-(L1-Pad1): track 4.56 -> 0.00 mm
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- removed copper zone on F.Cu, net GND
